File: UnoMiniC.kicad_sch (KiCad schematic)
At the start: 58 parts, among them J1 HDR-M-2.54_2x3, J2 HDR-M-2.54_2x3, J3 HDR-M-2.54_1x16, J4 HDR-M-2.54_1x16, Q1 DMG3415UQ-7, SW1 KMR221GLFS, U1.1 LM358DR, U1.2 LM358DR, U2 LD1117S33CTR, U3 LP2985IM5X-3.3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

Commit message: Updated Documentation
Parts:
- removed A: A, symbol Unknown_890_-1749
Other:
- moved on the sheet: C1, C10, C11, C12, C13, C2, C3, C4, C5, C6, C7, C8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
